File: BookerBoard v1.0/BookerBoard.kicad_pcb (KiCad board)
At the start: 2 copper layers, 189.7 x 77 mm, 34 parts, among them U1 ProMicro

Commit message: 5/3/20 v1
Routing:
- net col2: track 138.4 -> 137.5 mm
Other:
- outline, holes or cut-outs redrawn
